File: KW2CPU.PCB.sch (EAGLE design)
At the start: 58 parts, among them IC1 AT45DB161D8S1

Commit message: Labeled all nets
Named nets and simplified JTAG adapter board.
Connections:
- net CLKM1 renamed XTAL_32M
- net CLKM2 renamed EXTAL_32M
- net N$1 renamed TAMPER/!RTC_WAKEUP
- net N$10 renamed PTA0/JTAG_TCLK/SWD_CLK/EZP_CLK/!UART0_CTS/!UART0_COL/FTM0_CH5
- net N$11 renamed PTA1/JTAG_TDI/EZP_DI/UART0/RX/FTM0_CH6
- net N$12 renamed PTA2/JTAG_TDO/TRACE?SWO/EZP_DO/UART0_TX/FTM0_CH7
- net N$13 renamed PTA3/JTAG_TMS/SWD_DIO/UART0_RTS/FTM0_CH0
- net N$14 renamed !RESET
- net N$15 renamed PTA4/LLWU_P3/!NMI!/!EZP_CS!/FTM0_CH1
- net N$16 renamed PTC5/LLWU_P8/SPI0_PCS0/UART1_TX/FTM0_CH3/CMP1_OUT
- net N$17 renamed PTC6/LLWU_P10/CMP0_IN0/SPI0_SOUT/PDB0_EXTRG/I2S0_RX_BCLK/I2S0_MCLK
- net N$18 renamed PTC7/CMP0_IN1/SPI0_SIN/USB_SOF_OUT/I2S0_RX_FS
- net N$19 renamed RFN
- net N$2 renamed RF_OUTP
- net N$20 renamed RFP
- net N$21 renamed ANT1
- net N$22 renamed VCC_DIG_PA
- net N$23 renamed F_ANT
- net N$24 renamed ANT2
- net N$25 renamed MMCX_ANT
- net N$26 renamed ANT_A
- net N$27 renamed ANTSEL
- net N$28 renamed EXTAL32
- net N$29 renamed C_LNA
- net N$3 renamed RF_OUTN
- net N$30 renamed RX_SWITCH
- net N$31 renamed TX_SWITCH
- net N$32 renamed XTAL32
- net N$33 renamed PTD2/LLWU_P13/SPI0_SOUT/UART2_RX/I2C0_SDA/GPIO4_BSM_DATA
- net N$34 renamed PTD1/ADC0_SE5B/SPI0_SCK/!UART2_CTS
- net N$35 renamed PTD3/SPI0_SIN/UART2_TX/I2C0_SCL/GPIO5_BSM_CLK
- net N$36 renamed PTD4/LLWU_P14/MADC0_SE21/SPI0_PCS1/!UART0_RTS!/FTM0_CH4/EWM_IN/GPIO_BSM_FRAME
- net N$37 renamed PTD5/ADC0_SE6B/SPI0_PCS2/!UART0_CTS!/!UART0_COL!/FTM0_CH5/!EWM_OUT
- net N$38 renamed PTD6/LLWU_P15/ADC0_SE7B/SPI0_PCS3/UART0_RX/FTM0_CH6/FTM0_FLT0
- net N$39 renamed PTD7/MADC0_SE22/CMT_IRO/UART0_TX/FTM0_CH7/FTM0_FLT1
- net N$40 renamed PTE0/MADC0_SE10/SPI1_PCS1/UART1_TX/MTRACE_CLKOUT/I2C1_SDA/RTC_CLKOUT
- net N$41 renamed PTE1/LLWU_P0/MADC0_SE11/SPI1_SOUT/UART1_RX/MTRACE_D3/I2C1_SCL/SPI1_SIN
- net N$42 renamed PTE2/LLWU_P1/MADC0_DP1/SPI1_SCK/!UART1_CTS!/MTRACE_D2
- net N$43 renamed PTE3/MADC0_DM1/SPI1_SIN/!UART1_RTS!/MTRACE_D1/SPI1_SOUT
- net N$44 renamed PTE4/LLWU_P2/SPI1_PCS0/MTRACE_D0
- net N$45 renamed PTE16/ADC0_SE4A/SPI0_PCS0/UART2_TX/FTM_CLKIN0/FTM0_FLT3
- net N$46 renamed PTE17/ADC0_SE5A/SPI0_SCK/UART2_RX/FTM_CLKIN1/LPTMR0_ALT3
- net N$47 renamed PTE18/ADC0_SE6A/SPI0_SOUT/!UART2_CTS!/I2C0_SDA
- net N$48 renamed PTE19/ADC0_SE7A/SPI0_SIN/!UART2_RTS!/I2C0_SCL
- net N$49 renamed PTA18/EXTAL0/FTM0_FTL2_FTM_CLKIN0
- net N$50 renamed PTA19/XTAL0/FTM1_FLT0/FTM_CLKIN1/LPTMR0_ALT1
- net N$51 renamed !CS
- net N$52 renamed SCK
- net N$53 renamed SI
- net N$7 renamed PTC4/LLWU_P8/SPI0_PCS0/UART1_TX/FTM0_CH3/CMP1_OUT
Changed lines of the file:
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@@
 </busses>
 <nets>
-<net name="CLKM1" class="0">
+<net name="XTAL_32M" class="0">
 <segment>
 <pinref part="U$2" gate="G$1" pin="P$3"/>
@@
 </segment>
 </net>
-<net name="CLKM2" class="0">
+<net name="EXTAL_32M" class="0">
 <segment>
 <pinref part="U$2" gate="G$1" pin="P$1"/>
@@
 </segment>
 </net>
-<net name="N$1" class="0">
+<net name="TAMPER/!RTC_WAKEUP" class="0">
 <segment>
 <pinref part="U$1" gate="G$1" pin="TAMPER0/!RTC_WAKEUP"/>
@@
 </segment>
 </net>
-<net name="N$7" class="0">
+<net name="PTC4/LLWU_P8/SPI0_PCS0/UART1_TX/FTM0_CH3/CMP1_OUT" class="0">
 <segment>
 <pinref part="U$1" gate="G$1" pin="PTC4/LLWU_P8/SPI0_PCS0/UART1_TX/FTM0_CH3/CMP1_OUT"/>
@@
 </segment>
 </net>
-<net name="N$16" class="0">
+<net name="PTC5/LLWU_P8/SPI0_PCS0/UART1_TX/FTM0_CH3/CMP1_OUT" class="0">
 <segment>
 <pinref part="U$1" gate="G$1" pin="PTC5/LLWU_P8/SPI0_PCS0/UART1_TX/FTM0_CH3/CMP1_OUT"/>
@@
 </segment>
 </net>
-<net name="N$17" class="0">
+<net name="PTC6/LLWU_P10/CMP0_IN0/SPI0_SOUT/PDB0_EXTRG/I2S0_RX_BCLK/I2S0_MCLK" class="0">
 <segment>
 <pinref part="U$1" gate="G$1" pin="PTC6/LLWU_P10/CMP0_IN0/SPI0_SOUT/PDB0_EXTRG/I2S0_RX_BCLK/I2S0_MCLK"/>
@@
 </segment>
 </net>
-<net name="N$18" class="0">
+<net name="PTC7/CMP0_IN1/SPI0_SIN/USB_SOF_OUT/I2S0_RX_FS" class="0">
 <segment>
 <pinref part="U$1" gate="G$1" pin="PTC7/CMP0_IN1/SPI0_SIN/USB_SOF_OUT/I2S0_RX_FS"/>
@@
 </segment>
 </net>
-<net name="N$2" class="0">
+<net name="RF_OUTP" class="0">
 <segment>
 <pinref part="U$1" gate="G$1" pin="RF_OUTP"/>
@@
 </segment>
 </net>
-<net name="N$3" class="0">
+<net name="RF_OUTN" class="0">
 <segment>
 <pinref part="L$4" gate="G$1" pin="1"/>
@@
 </segment>
 </net>
-<net name="N$19" class="0">
+<net name="RFN" class="0">
 <segment>
 <pinref part="R$7" gate="G$1" pin="2"/>
@@
 </segment>
 </net>
-<net name="N$20" class="0">
+<net name="RFP" class="0">
 <segment>
 <pinref part="U$3" gate="G$1" pin="RFP"/>
@@
 </segment>
 </net>
-<net name="N$22" class="0">
+<net name="VCC_DIG_PA" class="0">
 <segment>
 <pinref part="U$3" gate="G$1" pin="VCC_DIG"/>
@@
 </segment>
 </net>
-<net name="N$21" class="0">
+<net name="ANT1" class="0">
 <segment>
 <pinref part="U$3" gate="G$1" pin="ANT1"/>
@@
 </segment>
 </net>
-<net name="N$23" class="0">
+<net name="F_ANT" class="0">
 <segment>
 <pinref part="L$14" gate="G$1" pin="2"/>
@@
 </segment>
 </net>
-<net name="N$24" class="0">
+<net name="ANT2" class="0">
 <segment>
 <pinref part="U$3" gate="G$1" pin="ANT2"/>
@@
 </segment>
 </net>
-<net name="N$25" class="0">
+<net name="MMCX_ANT" class="0">
 <segment>
 <pinref part="L$17" gate="G$1" pin="1"/>
@@
 </segment>
 </net>
-<net name="N$26" class="0">
+<net name="ANT_A" class="0">
 <segment>
 <pinref part="U$1" gate="G$1" pin="ANT_A"/>
@@
 </segment>
 </net>
-<net name="N$27" class="0">
+<net name="ANTSEL" class="0">
 <segment>
 <pinref part="R$19" gate="G$1" pin="1"/>
@@
 </segment>
 </net>
-<net name="N$31" class="0">
+<net name="TX_SWITCH" class="0">
 <segment>
 <pinref part="U$3" gate="G$1" pin="C_RX_TX"/>
@@
 </segment>
 </net>
-<net name="N$30" class="0">
+<net name="RX_SWITCH" class="0">
 <segment>
 <pinref part="C$24" gate="G$1" pin="1"/>
@@
 </segment>
 </net>
-<net name="N$28" class="0">
+<net name="EXTAL32" class="0">
 <segment>
 <pinref part="U$7" gate="G$1" pin="1"/>
@@
 </segment>
 </net>
-<net name="N$32" class="0">
+<net name="XTAL32" class="0">
 <segment>
 <pinref part="U$7" gate="G$1" pin="2"/>
@@
 </segment>
 </net>
-<net name="N$34" class="0">
+<net name="PTD1/ADC0_SE5B/SPI0_SCK/!UART2_CTS" class="0">
 <segment>
 <pinref part="U$1" gate="G$1" pin="PTD1/ADC0_SE5B/SPI0_SCK/!UART2_CTS"/>
@@
 </segment>
 </net>
-<net name="N$33" class="0">
+<net name="PTD2/LLWU_P13/SPI0_SOUT/UART2_RX/I2C0_SDA/GPIO4_BSM_DATA" class="0">
 <segment>
 <pinref part="U$1" gate="G$1" pin="PTD2/LLWU_P13/SPI0_SOUT/UART2_RX/I2C0_SDA/GPIO4_BSM_DATA"/>
@@
 </segment>
 </net>
-<net name="N$35" class="0">
+<net name="PTD3/SPI0_SIN/UART2_TX/I2C0_SCL/GPIO5_BSM_CLK" class="0">
 <segment>
 <pinref part="U$1" gate="G$1" pin="PTD3/SPI0_SIN/UART2_TX/I2C0_SCL/GPIO5_BSM_CLK"/>
@@
 </segment>
 </net>
-<net name="N$36" class="0">
+<net name="PTD4/LLWU_P14/MADC0_SE21/SPI0_PCS1/!UART0_RTS!/FTM0_CH4/EWM_IN/GPIO_BSM_FRAME" class="0">
 <segment>
 <pinref part="U$1" gate="G$1" pin="PTD4/LLWU_P14/MADC0_SE21/SPI0_PCS1/!UART0_RTS!/FTM0_CH4/EWM_IN/GPIO_BSM_FRAME"/>
@@
 </segment>
 </net>
-<net name="N$37" class="0">
+<net name="PTD5/ADC0_SE6B/SPI0_PCS2/!UART0_CTS!/!UART0_COL!/FTM0_CH5/!EWM_OUT" class="0">
 <segment>
 <pinref part="U$1" gate="G$1" pin="PTD5/ADC0_SE6B/SPI0_PCS2/!UART0_CTS!/!UART0_COL!/FTM0_CH5/!EWM_OUT"/>
@@
 </segment>
 </net>
-<net name="N$38" class="0">
+<net name="PTD6/LLWU_P15/ADC0_SE7B/SPI0_PCS3/UART0_RX/FTM0_CH6/FTM0_FLT0" class="0">
 <segment>
 <pinref part="U$1" gate="G$1" pin="PTD6/LLWU_P15/ADC0_SE7B/SPI0_PCS3/UART0_RX/FTM0_CH6/FTM0_FLT0"/>
@@
 </segment>
 </net>
-<net name="N$39" class="0">
+<net name="PTD7/MADC0_SE22/CMT_IRO/UART0_TX/FTM0_CH7/FTM0_FLT1" class="0">
 <segment>
 <pinref part="U$1" gate="G$1" pin="PTD7/MADC0_SE22/CMT_IRO/UART0_TX/FTM0_CH7/FTM0_FLT1"/>
@@
 </segment>
 </net>
-<net name="N$40" class="0">
+<net name="PTE0/MADC0_SE10/SPI1_PCS1/UART1_TX/MTRACE_CLKOUT/I2C1_SDA/RTC_CLKOUT" class="0">
 <segment>
 <pinref part="U$1" gate="G$1" pin="PTE0/MADC0_SE10/SPI1_PCS1/UART1_TX/MTRACE_CLKOUT/I2C1_SDA/RTC_CLKOUT"/>
@@
 </segment>
 </net>
-<net name="N$41" class="0">
+<net name="PTE1/LLWU_P0/MADC0_SE11/SPI1_SOUT/UART1_RX/MTRACE_D3/I2C1_SCL/SPI1_SIN" class="0">
 <segment>
 <pinref part="U$1" gate="G$1" pin="PTE1/LLWU_P0/MADC0_SE11/SPI1_SOUT/UART1_RX/MTRACE_D3/I2C1_SCL/SPI1_SIN"/>
@@
 </segment>
 </net>
-<net name="N$42" class="0">
+<net name="PTE2/LLWU_P1/MADC0_DP1/SPI1_SCK/!UART1_CTS!/MTRACE_D2" class="0">
 <segment>
 <pinref part="U$1" gate="G$1" pin="PTE2/LLWU_P1/MADC0_DP1/SPI1_SCK/!UART1_CTS!/MTRACE_D2"/>
@@
 </segment>
 </net>
-<net name="N$43" class="0">
+<net name="PTE3/MADC0_DM1/SPI1_SIN/!UART1_RTS!/MTRACE_D1/SPI1_SOUT" class="0">
 <segment>
 <pinref part="U$1" gate="G$1" pin="PTE3/MADC0_DM1/SPI1_SIN/!UART1_RTS!/MTRACE_D1/SPI1_SOUT"/>
@@
 </segment>
 </net>
-<net name="N$44" class="0">
+<net name="PTE4/LLWU_P2/SPI1_PCS0/MTRACE_D0" class="0">
 <segment>
 <pinref part="U$1" gate="G$1" pin="PTE4/LLWU_P2/SPI1_PCS0/MTRACE_D0"/>
@@
 </segment>
 </net>
-<net name="N$45" class="0">
+<net name="PTE16/ADC0_SE4A/SPI0_PCS0/UART2_TX/FTM_CLKIN0/FTM0_FLT3" class="0">
 <segment>
 <pinref part="U$1" gate="G$1" pin="PTE16/ADC0_SE4A/SPI0_PCS0/UART2_TX/FTM_CLKIN0/FTM0_FLT3"/>
@@
 </segment>
 </net>
-<net name="N$46" class="0">
+<net name="PTE17/ADC0_SE5A/SPI0_SCK/UART2_RX/FTM_CLKIN1/LPTMR0_ALT3" class="0">
 <segment>
 <pinref part="U$1" gate="G$1" pin="PTE17/ADC0_SE5A/SPI0_SCK/UART2_RX/FTM_CLKIN1/LPTMR0_ALT3"/>
@@
 </segment>
 </net>
-<net name="N$47" class="0">
+<net name="PTE18/ADC0_SE6A/SPI0_SOUT/!UART2_CTS!/I2C0_SDA" class="0">
 <segment>
 <pinref part="U$1" gate="G$1" pin="PTE18/ADC0_SE6A/SPI0_SOUT/!UART2_CTS!/I2C0_SDA"/>
@@
 </segment>
 </net>
-<net name="N$10" class="0">
+<net name="PTA0/JTAG_TCLK/SWD_CLK/EZP_CLK/!UART0_CTS/!UART0_COL/FTM0_CH5" class="0">
 <segment>
 <pinref part="U$1" gate="G$1" pin="PTA0/JTAG_TCLK/SWD_CLK/EZP_CLK/!UART0_CTS/!UART0_COL/FTM0_CH5"/>
@@
 </segment>
 </net>
-<net name="N$11" class="0">
+<net name="PTA1/JTAG_TDI/EZP_DI/UART0/RX/FTM0_CH6" class="0">
 <segment>
 <pinref part="U$1" gate="G$1" pin="PTA1/JTAG_TDI/EZP_DI/UART0/RX/FTM0_CH6"/>
@@
 </segment>
 </net>
-<net name="N$12" class="0">
+<net name="PTA2/JTAG_TDO/TRACE?SWO/EZP_DO/UART0_TX/FTM0_CH7" class="0">
 <segment>
 <pinref part="U$1" gate="G$1" pin="PTA2/JTAG_TDO/TRACE?SWO/EZP_DO/UART0_TX/FTM0_CH7"/>
@@
 </segment>
 </net>
-<net name="N$13" class="0">
+<net name="PTA3/JTAG_TMS/SWD_DIO/UART0_RTS/FTM0_CH0" class="0">
 <segment>
 <pinref part="U$1" gate="G$1" pin="PTA3/JTAG_TMS/SWD_DIO/UART0_RTS/FTM0_CH0"/>
@@
 </segment>
 </net>
-<net name="N$15" class="0">
+<net name="PTA4/LLWU_P3/!NMI!/!EZP_CS!/FTM0_CH1" class="0">
 <segment>
 <pinref part="U$1" gate="G$1" pin="PTA4/LLWU_P3/!NMI!/!EZP_CS!/FTM0_CH1"/>
@@
 </segment>
 </net>
-<net name="N$49" class="0">
+<net name="PTA18/EXTAL0/FTM0_FTL2_FTM_CLKIN0" class="0">
 <segment>
 <pinref part="U$1" gate="G$1" pin="PTA18/EXTAL0/FTM0_FTL2_FTM_CLKIN0"/>
@@
 </segment>
 </net>
-<net name="N$50" class="0">
+<net name="PTA19/XTAL0/FTM1_FLT0/FTM_CLKIN1/LPTMR0_ALT1" class="0">
 <segment>
 <pinref part="U$1" gate="G$1" pin="PTA19/XTAL0/FTM1_FLT0/FTM_CLKIN1/LPTMR0_ALT1"/>
@@
 </segment>
 </net>
-<net name="N$48" class="0">
+<net name="PTE19/ADC0_SE7A/SPI0_SIN/!UART2_RTS!/I2C0_SCL" class="0">
 <segment>
 <pinref part="U$1" gate="G$1" pin="PTE19/ADC0_SE7A/SPI0_SIN/!UART2_RTS!/I2C0_SCL"/>
@@
 </segment>
 </net>
-<net name="N$14" class="0">
+<net name="!RESET" class="0">
 <segment>
 <pinref part="U$1" gate="G$1" pin="!RESET"/>
@@
 </segment>
 </net>
-<net name="N$29" class="0">
+<net name="C_LNA" class="0">
 <segment>
 <pinref part="R$1" gate="G$1" pin="1"/>
@@
 </segment>
 </net>
-<net name="N$51" class="0">
+<net name="!CS" class="0">
 <segment>
 <pinref part="IC1" gate="G$1" pin="!CS"/>
@@
 <pinref part="U$8" gate="G$1" pin="1"/>
 <wire x1="-76.2" y1="-93.98" x2="-76.2" y2="-55.88" width="0.1524" layer="91"/>
-</segment>
-</net>
-<net name="N$52" class="0">
+<label x="-110.49" y="-92.71" size="1.778" layer="95"/>
+</segment>
+</net>
+<net name="SCK" class="0">
 <segment>
 <pinref part="IC1" gate="G$1" pin="SCK"/>
@@
 </segment>
 </net>
-<net name="N$53" class="0">
+<net name="SI" class="0">
 <segment>
 <pinref part="IC1" gate="G$1" pin="SI"/>

Commit message: Fixed RefDes, issues with names disappearing
Names on layout disappearing (for RF front end parts)
Parts:
- renumbered C$10 to C23, C$13 to C25, C$15 to C24, C$16 to C27, C$18 to C26, C$20 to C28, C$21 to C29, C$22 to C30, C$24 to C21, C$6 to C20, C$9 to C22, IC1 to U2, IC2 to U4, L$11 to L3, L$14 to L4, L$17 to L5, L$4 to L1, L$5 to L2, R$1 to R7, R$19 to R9, R$2 to R8, R$23 to R6, R$7 to R4, R$8 to R5, U$1 to U1, U$10 to JP3, U$11 to JP4, U$12 to J2, U$2 to X2, U$3 to U3, U$4 to U5, U$5 to J3, U$6 to J1, U$7 to X1, U$8 to JP1, U$9 to JP2
