File: KW2CPU.PCB Design Files/JTAG.sch (EAGLE design)
At the start: 2 parts

Commit message: Added part numbers and manufacturers (inconsistent)
Also moved files to proper directories. Needs manual inconsistency
fixing
Parts:
- U$1: MFGN (none) -> MOLEX; MFGP (none) -> 54722-0304
Changed lines of the file:
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@@
 </classes>
 <parts>
-<part name="U$1" library="KW2" deviceset="MOLEX54722-0304" device=""/>
+<part name="U$1" library="KW2" deviceset="MOLEX54722-0304" device="">
+<attribute name="MFGN" value="MOLEX"/>
+<attribute name="MFGP" value="54722-0304"/>
+</part>
 <part name="U$2" library="KW2" deviceset="2X10JTAG" device=""/>
 </parts>
@@
 </plain>
 <instances>
-<instance part="U$1" gate="G$1" x="0" y="-10.16" rot="MR270"/>
+<instance part="U$1" gate="G$1" x="0" y="-10.16" rot="MR270">
+<attribute name="MFGN" x="0" y="-10.16" size="1.778" layer="96" rot="MR270" display="off"/>
+<attribute name="MFGP" x="0" y="-10.16" size="1.778" layer="96" rot="MR270" display="off"/>
+</instance>
 <instance part="U$2" gate="G$1" x="55.88" y="-10.16" rot="R270"/>
 </instances>
