File: KW2CPU.PCB Design Files/KW2CPU.PCB.sch (EAGLE design)
At the start: 81 parts, among them IC1 25AA080SN, J1 DF12_M, U1 MKW21D, U3 RF6555, X1 32KHZ, X2 32MHZ

Commit message: Connect RF6555 CE to KW2 AREG
Connections:
- removed net N$6: C5.1, C6.1, C7.1, U1.VDD_IF, U1.VDD_PA, U1.VDD_RF
- removed net RX_SWITCH: C21.1, R6.1, TP7.TP, U1.RX_SWITCH, U3.CE
- new net RADIO_AREG: C21.1, C5.1, C6.1, C7.1, R6.1, TP7.TP, U1.VDD_IF, U1.VDD_PA, U1.VDD_RF, U3.CE
Other:
- moved on the sheet: C16, C17, C18
Changed lines of the file:
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@@
 <attribute name="MFGP" x="-88.9" y="78.74" size="1.778" layer="96" display="off"/>
 </instance>
-<instance part="C16" gate="G$1" x="40.64" y="78.74">
-<attribute name="MFGN" x="40.64" y="78.74" size="1.778" layer="96" display="off"/>
-<attribute name="MFGP" x="40.64" y="78.74" size="1.778" layer="96" display="off"/>
-</instance>
-<instance part="C17" gate="G$1" x="30.48" y="78.74">
-<attribute name="MFGN" x="30.48" y="78.74" size="1.778" layer="96" display="off"/>
-<attribute name="MFGP" x="30.48" y="78.74" size="1.778" layer="96" display="off"/>
-</instance>
-<instance part="C18" gate="G$1" x="20.32" y="78.74">
-<attribute name="MFGN" x="20.32" y="78.74" size="1.778" layer="96" display="off"/>
-<attribute name="MFGP" x="20.32" y="78.74" size="1.778" layer="96" display="off"/>
+<instance part="C16" gate="G$1" x="48.26" y="78.74">
+<attribute name="MFGN" x="48.26" y="78.74" size="1.778" layer="96" display="off"/>
+<attribute name="MFGP" x="48.26" y="78.74" size="1.778" layer="96" display="off"/>
+</instance>
+<instance part="C17" gate="G$1" x="38.1" y="78.74">
+<attribute name="MFGN" x="38.1" y="78.74" size="1.778" layer="96" display="off"/>
+<attribute name="MFGP" x="38.1" y="78.74" size="1.778" layer="96" display="off"/>
+</instance>
+<instance part="C18" gate="G$1" x="27.94" y="78.74">
+<attribute name="MFGN" x="27.94" y="78.74" size="1.778" layer="96" display="off"/>
+<attribute name="MFGP" x="27.94" y="78.74" size="1.778" layer="96" display="off"/>
 </instance>
 <instance part="GND5" gate="1" x="-10.16" y="93.98"/>
-<instance part="GND8" gate="1" x="30.48" y="71.12"/>
+<instance part="GND8" gate="1" x="38.1" y="71.12"/>
 <instance part="GND9" gate="1" x="-78.74" y="71.12"/>
 <instance part="GND10" gate="1" x="-17.78" y="58.42"/>
 <instance part="+3V2" gate="G$1" x="-45.72" y="86.36"/>
 <instance part="+3V3" gate="G$1" x="-78.74" y="86.36"/>
-<instance part="+3V4" gate="G$1" x="30.48" y="88.9"/>
+<instance part="+3V4" gate="G$1" x="38.1" y="88.9"/>
 <instance part="GND11" gate="1" x="-91.44" y="25.4"/>
-<instance part="+3V5" gate="G$1" x="15.24" y="68.58"/>
+<instance part="+3V5" gate="G$1" x="15.24" y="66.04"/>
 <instance part="R1" gate="G$1" x="-116.84" y="12.7">
 <attribute name="MFGN" x="-116.84" y="12.7" size="1.778" layer="96" display="off"/>
@@
 <wire x1="-68.58" y1="25.4" x2="-66.04" y2="25.4" width="0.1524" layer="91"/>
 <junction x="-88.9" y="40.64"/>
-</segment>
-</net>
-<net name="N$6" class="0">
-<segment>
-<pinref part="U1" gate="G$1" pin="VDD_RF"/>
-<wire x1="-5.08" y1="55.88" x2="-5.08" y2="60.96" width="0.1524" layer="91"/>
-<pinref part="U1" gate="G$1" pin="VDD_IF"/>
-<wire x1="-5.08" y1="60.96" x2="-7.62" y2="60.96" width="0.1524" layer="91"/>
-<wire x1="-7.62" y1="60.96" x2="-7.62" y2="55.88" width="0.1524" layer="91"/>
-<pinref part="U1" gate="G$1" pin="VDD_PA"/>
-<wire x1="-7.62" y1="60.96" x2="-10.16" y2="60.96" width="0.1524" layer="91"/>
-<wire x1="-10.16" y1="60.96" x2="-10.16" y2="55.88" width="0.1524" layer="91"/>
-<junction x="-7.62" y="60.96"/>
-<pinref part="C7" gate="G$1" pin="1"/>
-<wire x1="-7.62" y1="73.66" x2="-17.78" y2="73.66" width="0.1524" layer="91"/>
-<pinref part="C6" gate="G$1" pin="1"/>
-<junction x="-7.62" y="73.66"/>
-<wire x1="-7.62" y1="60.96" x2="-7.62" y2="73.66" width="0.1524" layer="91"/>
-<junction x="-7.62" y="73.66"/>
-<pinref part="C5" gate="G$1" pin="1"/>
-<wire x1="-7.62" y1="73.66" x2="2.54" y2="73.66" width="0.1524" layer="91"/>
 </segment>
 </net>
@@
 <pinref part="C18" gate="G$1" pin="1"/>
 <pinref part="C17" gate="G$1" pin="1"/>
-<wire x1="20.32" y1="81.28" x2="30.48" y2="81.28" width="0.1524" layer="91"/>
+<wire x1="27.94" y1="81.28" x2="38.1" y2="81.28" width="0.1524" layer="91"/>
 <pinref part="C16" gate="G$1" pin="1"/>
-<wire x1="30.48" y1="81.28" x2="40.64" y2="81.28" width="0.1524" layer="91"/>
-<junction x="30.48" y="81.28"/>
+<wire x1="38.1" y1="81.28" x2="48.26" y2="81.28" width="0.1524" layer="91"/>
+<junction x="38.1" y="81.28"/>
 <pinref part="U1" gate="G$1" pin="VBAT_RF"/>
 <wire x1="7.62" y1="55.88" x2="7.62" y2="63.5" width="0.1524" layer="91"/>
-<junction x="20.32" y="81.28"/>
+<junction x="27.94" y="81.28"/>
 <pinref part="U1" gate="G$1" pin="VBAT2_RF"/>
-<wire x1="7.62" y1="81.28" x2="20.32" y2="81.28" width="0.1524" layer="91"/>
+<wire x1="22.86" y1="81.28" x2="27.94" y2="81.28" width="0.1524" layer="91"/>
 <wire x1="5.08" y1="55.88" x2="5.08" y2="63.5" width="0.1524" layer="91"/>
 <wire x1="5.08" y1="63.5" x2="7.62" y2="63.5" width="0.1524" layer="91"/>
 <junction x="7.62" y="63.5"/>
-<wire x1="7.62" y1="81.28" x2="7.62" y2="63.5" width="0.1524" layer="91"/>
-<junction x="7.62" y="81.28"/>
 <pinref part="+3V4" gate="G$1" pin="+3V3"/>
-<wire x1="30.48" y1="81.28" x2="30.48" y2="86.36" width="0.1524" layer="91"/>
+<wire x1="7.62" y1="68.58" x2="7.62" y2="63.5" width="0.1524" layer="91"/>
+<wire x1="38.1" y1="81.28" x2="38.1" y2="86.36" width="0.1524" layer="91"/>
+<wire x1="7.62" y1="68.58" x2="22.86" y2="68.58" width="0.1524" layer="91"/>
+<wire x1="22.86" y1="68.58" x2="22.86" y2="81.28" width="0.1524" layer="91"/>
 </segment>
 <segment>
@@
 <wire x1="15.24" y1="63.5" x2="15.24" y2="55.88" width="0.1524" layer="91"/>
 <pinref part="+3V5" gate="G$1" pin="+3V3"/>
-<wire x1="15.24" y1="63.5" x2="15.24" y2="66.04" width="0.1524" layer="91"/>
 </segment>
 <segment>
@@
 </segment>
 </net>
-<net name="RX_SWITCH" class="0">
+<net name="RADIO_AREG" class="0">
 <segment>
 <pinref part="C21" gate="G$1" pin="1"/>
@@
 <wire x1="271.78" y1="2.54" x2="271.78" y2="96.52" width="0.1524" layer="91"/>
 <wire x1="271.78" y1="96.52" x2="271.78" y2="116.84" width="0.1524" layer="91"/>
-<wire x1="271.78" y1="116.84" x2="-154.94" y2="116.84" width="0.1524" layer="91"/>
-<wire x1="-154.94" y1="116.84" x2="-154.94" y2="-2.54" width="0.1524" layer="91"/>
-<wire x1="-154.94" y1="-2.54" x2="-129.54" y2="-2.54" width="0.1524" layer="91"/>
-<wire x1="-129.54" y1="-2.54" x2="-129.54" y2="0" width="0.1524" layer="91"/>
-<pinref part="U1" gate="G$1" pin="RX_SWITCH"/>
-<wire x1="-129.54" y1="0" x2="-66.04" y2="0" width="0.1524" layer="91"/>
+<wire x1="271.78" y1="116.84" x2="17.78" y2="116.84" width="0.1524" layer="91"/>
 <pinref part="TP7" gate="G$1" pin="TP"/>
 <wire x1="292.1" y1="104.14" x2="292.1" y2="96.52" width="0.1524" layer="91"/>
@@
 <junction x="289.56" y="2.54"/>
 <junction x="299.72" y="2.54"/>
+<pinref part="U1" gate="G$1" pin="VDD_RF"/>
+<wire x1="-5.08" y1="55.88" x2="-5.08" y2="60.96" width="0.1524" layer="91"/>
+<pinref part="U1" gate="G$1" pin="VDD_IF"/>
+<wire x1="-5.08" y1="60.96" x2="-7.62" y2="60.96" width="0.1524" layer="91"/>
+<wire x1="-7.62" y1="60.96" x2="-7.62" y2="55.88" width="0.1524" layer="91"/>
+<pinref part="U1" gate="G$1" pin="VDD_PA"/>
+<wire x1="-7.62" y1="60.96" x2="-10.16" y2="60.96" width="0.1524" layer="91"/>
+<wire x1="-10.16" y1="60.96" x2="-10.16" y2="55.88" width="0.1524" layer="91"/>
+<junction x="-7.62" y="60.96"/>
+<pinref part="C7" gate="G$1" pin="1"/>
+<wire x1="-7.62" y1="73.66" x2="-17.78" y2="73.66" width="0.1524" layer="91"/>
+<pinref part="C6" gate="G$1" pin="1"/>
+<junction x="-7.62" y="73.66"/>
+<wire x1="-7.62" y1="60.96" x2="-7.62" y2="71.12" width="0.1524" layer="91"/>
+<junction x="-7.62" y="73.66"/>
+<pinref part="C5" gate="G$1" pin="1"/>
+<wire x1="-7.62" y1="71.12" x2="-7.62" y2="73.66" width="0.1524" layer="91"/>
+<wire x1="-7.62" y1="73.66" x2="2.54" y2="73.66" width="0.1524" layer="91"/>
+<wire x1="-7.62" y1="71.12" x2="17.78" y2="71.12" width="0.1524" layer="91"/>
+<wire x1="17.78" y1="71.12" x2="17.78" y2="116.84" width="0.1524" layer="91"/>
+<junction x="-7.62" y="71.12"/>
 </segment>
 </net>
@@
 <pinref part="C18" gate="G$1" pin="2"/>
 <pinref part="C17" gate="G$1" pin="2"/>
-<wire x1="20.32" y1="73.66" x2="30.48" y2="73.66" width="0.1524" layer="91"/>
+<wire x1="27.94" y1="73.66" x2="38.1" y2="73.66" width="0.1524" layer="91"/>
 <pinref part="C16" gate="G$1" pin="2"/>
-<wire x1="40.64" y1="73.66" x2="30.48" y2="73.66" width="0.1524" layer="91"/>
-<junction x="30.48" y="73.66"/>
+<wire x1="48.26" y1="73.66" x2="38.1" y2="73.66" width="0.1524" layer="91"/>
+<junction x="38.1" y="73.66"/>
 <pinref part="GND8" gate="1" pin="GND"/>
 </segment>
